Commit message: Update rviz visualization

File: catkin_ws/src/arena_mapping/assets/urdf/minibot.urdf (robot description, URDF)
Before this commit: robot minibot, 1 links, 0 joints
Links:
- added link aruco_marker; visual box size=0.1 0.1 0.001
Joints:
- added joint aruco_to_base: type fixed, parent base_link, child aruco_marker, origin xyz=0 0 0.12 rpy=0 0 0
