Commit message: Add hardware pkg simul

File: catkin_ws/src/simulator_physics/mobile_base/assets/urdf/minibot.urdf (robot description, URDF)
Before this commit: robot minibot, 2 links, 1 joints
Links:
- added link laser_link; visual cylinder length=0.05 radius=0.01
Joints:
- added joint laser_to_base: type fixed, parent base_link, child laser_link, origin xyz=0 0 0.12 rpy=0 0 0
